File: Power.kicad_sch (KiCad schematic)
At the start: 28 parts

Commit message: Add files via upload
Other:
- moved on the sheet: C17, U2

Commit message: Add files via upload
Other:
- moved on the sheet: C17, U2
