File: boot.kicad_sch (KiCad schematic)
At the start: 1 part

Commit message: Add files via upload
Connections:
- net DAT3/CD is gone; now on net GND: U?.2 (DAT3/CD)
Changed lines of the file:
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@@
-	(wire
-		(pts
-			(xy 181.61 78.74) (xy 190.5 78.74)
-		)
-		(stroke
-			(width 0)
-			(type default)
-		)
-	)
 	(wire
 		(pts
@@
 	(wire
 		(pts
+			(xy 100.33 88.9) (xy 121.92 88.9)
+		)
+		(stroke
+			(width 0)
+			(type default)
+		)
+	)
+	(wire
+		(pts
 			(xy 106.68 80.01) (xy 106.68 93.98)
 		)
@@
 		)
 	)
-	(global_label "DAT3{slash}CD"
-		(shape input)
-		(at 181.61 78.74 180)
-		(fields_autoplaced yes)
-		(effects
-			(font
-				(size 1.27 1.27)
-			)
-			(justify right)
-		)
-		(property "Intersheetrefs" "${INTERSHEET_REFS}"
-			(at 170.2186 78.74 0)
-			(effects
-				(font
-					(size 1.27 1.27)
-				)
-				(justify right)
-				(hide yes)
-			)
-		)
-	)
 	(global_label "DAT0"
 		(shape input)
@@
 		)
 	)
-	(global_label "DAT3{slash}CD"
-		(shape input)
-		(at 121.92 88.9 180)
-		(fields_autoplaced yes)
-		(effects
-			(font
-				(size 1.27 1.27)
-			)
-			(justify right)
-		)
-		(property "Intersheetrefs" "${INTERSHEET_REFS}"
-			(at 110.5286 88.9 0)
-			(effects
-				(font
-					(size 1.27 1.27)
-				)
-				(justify right)
-				(hide yes)
-			)
-		)
-	)
 	(global_label "CMD"
 		(shape input)
@@
 		(shape input)
 		(at 190.5 83.82 0)
-		(fields_autoplaced yes)
 		(effects
 			(font
@@
 		(shape input)
 		(at 190.5 74.93 0)
-		(fields_autoplaced yes)
 		(effects
 			(font
@@
 		(shape input)
 		(at 190.5 99.06 0)
-		(fields_autoplaced yes)
 		(effects
 			(font
@@
 		(shape input)
 		(at 190.5 88.9 0)
-		(fields_autoplaced yes)
 		(effects
 			(font
@@
 		)
 	)
-	(hierarchical_label "DAT3{slash}CD"
-		(shape input)
-		(at 190.5 78.74 0)
-		(fields_autoplaced yes)
-		(effects
-			(font
-				(size 1.27 1.27)
-			)
-			(justify left)
-		)
-	)
 	(hierarchical_label "DAT0"
 		(shape input)
 		(at 190.5 93.98 0)
-		(fields_autoplaced yes)
 		(effects
 			(font
@@
 		(instances
 			(project ""
-				(path "/5516d47b-e414-41cc-be39-f34e0b8598e1/8cf1266b-f0c8-4bea-b6a6-3602ef8d967e"
+				(path "/5516d47b-e414-41cc-be39-f34e0b8598e1/c1572ada-486c-48b1-b220-bdb459cea861"
 					(reference "U?")
+					(unit 1)
+				)
+			)
+		)
+	)
+	(symbol
+		(lib_id "power:GND")
+		(at 100.33 88.9 0)
+		(unit 1)
+		(exclude_from_sim no)
+		(in_bom yes)
+		(on_board yes)
+		(dnp no)
+		(fields_autoplaced yes)
+		(property "Reference" "#PWR031"
+			(at 100.33 95.25 0)
+			(effects
+				(font
+					(size 1.27 1.27)
+				)
+				(hide yes)
+			)
+		)
+		(property "Value" "GND"
+			(at 100.33 93.98 0)
+			(effects
+				(font
+					(size 1.27 1.27)
+				)
+			)
+		)
+		(property "Footprint" ""
+			(at 100.33 88.9 0)
+			(effects
+				(font
+					(size 1.27 1.27)
+				)
+				(hide yes)
+			)
+		)
+		(property "Datasheet" ""
+			(at 100.33 88.9 0)
+			(effects
+				(font
+					(size 1.27 1.27)
+				)
+				(hide yes)
+			)
+		)
+		(property "Description" "Power symbol creates a global label with name \"GND\" , ground"
+			(at 100.33 88.9 0)
+			(effects
+				(font
+					(size 1.27 1.27)
+				)
+				(hide yes)
+			)
+		)
+		(pin "1"
+		)
+		(instances
+			(project ""
+				(path "/5516d47b-e414-41cc-be39-f34e0b8598e1/c1572ada-486c-48b1-b220-bdb459cea861"
+					(reference "#PWR031")
 					(unit 1)
 				)
@@
 		(instances
 			(project ""
-				(path "/5516d47b-e414-41cc-be39-f34e0b8598e1/8cf1266b-f0c8-4bea-b6a6-3602ef8d967e"
+				(path "/5516d47b-e414-41cc-be39-f34e0b8598e1/c1572ada-486c-48b1-b220-bdb459cea861"
 					(reference "#PWR033")
 					(unit 1)
@@
 		(instances
 			(project ""
-				(path "/5516d47b-e414-41cc-be39-f34e0b8598e1/8cf1266b-f0c8-4bea-b6a6-3602ef8d967e"
+				(path "/5516d47b-e414-41cc-be39-f34e0b8598e1/c1572ada-486c-48b1-b220-bdb459cea861"
 					(reference "#PWR032")
 					(unit 1)

Commit message: Add files via upload
Parts:
- removed U?: ~, symbol Aftx07:MSD-4-A
- added U?: ~, symbol Aftx07:MSD-4-A
Connections:
- net +3.3V: now also U?.4 (VDD)
- net CLK: now also U?.5 (CLK)
- net CMD: now also U?.3 (CMD)
- net DAT0: now also U?.7 (DAT0)
- net DAT1: now also U?.8 (DAT1)
- net DAT2: now also U?.1 (DAT2)
- net GND: now also U?.6 (VSS)
- new net DAT3/CD: U?.2 (DAT3/CD)
